File: circuit/kicad/sheet_beam_peltier.kicad_sch (KiCad schematic)
At the start: 3 parts, among them J701 Beam_PWM_Inputs, J702 RGB_Load_Out, J703 Peltier_Load_Out

Commit message: Refactor controller roles and update power/resistor schematics
Parts:
- added R701, R702, R703: 1R, symbol Device:R
Changed lines of the file:
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@@
+    (pin "2")
+  )
+  (symbol (lib_id "Device:R") (at 74 92.19 0) (unit 1)
+    (in_bom yes) (on_board yes)
+    (property "Reference" "R701" (id 0) (at 74 89.65 0))
+    (property "Value" "1R" (id 1) (at 74 94.73 0))
+    (property "Footprint" "" (id 2) (at 74 92.19 0)
+      (effects (font (size 1.27 1.27)) hide)
+    )
+    (property "Datasheet" "" (id 3) (at 74 92.19 0)
+      (effects (font (size 1.27 1.27)) hide)
+    )
+    (pin "1")
+    (pin "2")
+  )
+  (symbol (lib_id "Device:R") (at 74 94.73 0) (unit 1)
+    (in_bom yes) (on_board yes)
+    (property "Reference" "R702" (id 0) (at 74 92.19 0))
+    (property "Value" "1R" (id 1) (at 74 97.27 0))
+    (property "Footprint" "" (id 2) (at 74 94.73 0)
+      (effects (font (size 1.27 1.27)) hide)
+    )
+    (property "Datasheet" "" (id 3) (at 74 94.73 0)
+      (effects (font (size 1.27 1.27)) hide)
+    )
+    (pin "1")
+    (pin "2")
+  )
+  (symbol (lib_id "Device:R") (at 74 97.27 0) (unit 1)
+    (in_bom yes) (on_board yes)
+    (property "Reference" "R703" (id 0) (at 74 94.73 0))
+    (property "Value" "1R" (id 1) (at 74 99.81 0))
+    (property "Footprint" "" (id 2) (at 74 97.27 0)
+      (effects (font (size 1.27 1.27)) hide)
+    )
+    (property "Datasheet" "" (id 3) (at 74 97.27 0)
+      (effects (font (size 1.27 1.27)) hide)
+    )
+    (pin "1")
     (pin "2")
   )
@@
       (reference "J703") (unit 1) (value "Peltier_Load_Out") (footprint "Adafruit_Eagle:JST-PH-2-THM")
     )
+    (path "/0459a7f8-2ca2-4539-b326-d3ceb5aab69f"
+      (reference "R701") (unit 1) (value "1R") (footprint "")
+    )
+    (path "/9719f36e-d8f1-4feb-afcf-95f4de9033ce"
+      (reference "R702") (unit 1) (value "1R") (footprint "")
+    )
+    (path "/36d20e64-42bc-4b8c-b574-dd32f6ce2f85"
+      (reference "R703") (unit 1) (value "1R") (footprint "")
+    )
   )
