File: circuit/kicad/sheet_beam_peltier.kicad_sch (KiCad schematic)
At the start: 6 parts, among them J701 Beam_PWM_Inputs, J702 RGB_Load_Out, J703 Peltier_Load_Out

Commit message: Assign standard SMD footprints to resistors and fuses
Parts:
- R701, R702, R703: footprint (none) -> Resistor_SMD:R_0805_2012Metric
Changed lines of the file:
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@@
     (property "Reference" "R701" (id 0) (at 74 89.65 0))
     (property "Value" "1R" (id 1) (at 74 94.73 0))
-    (property "Footprint" "" (id 2) (at 74 92.19 0)
+    (property "Footprint" "Resistor_SMD:R_0805_2012Metric" (id 2) (at 74 92.19 0)
       (effects (font (size 1.27 1.27)) hide)
     )
@@
     (property "Reference" "R702" (id 0) (at 74 92.19 0))
     (property "Value" "1R" (id 1) (at 74 97.27 0))
-    (property "Footprint" "" (id 2) (at 74 94.73 0)
+    (property "Footprint" "Resistor_SMD:R_0805_2012Metric" (id 2) (at 74 94.73 0)
       (effects (font (size 1.27 1.27)) hide)
     )
@@
     (property "Reference" "R703" (id 0) (at 74 94.73 0))
     (property "Value" "1R" (id 1) (at 74 99.81 0))
-    (property "Footprint" "" (id 2) (at 74 97.27 0)
+    (property "Footprint" "Resistor_SMD:R_0805_2012Metric" (id 2) (at 74 97.27 0)
       (effects (font (size 1.27 1.27)) hide)
     )

Commit message: Migrate Orciny device to single-strip core and GPIO pump control
Replace the M0 NeoPXL8-based core controller with a single 30-pixel NeoPixel strip on D13 and keep Serial1 TX dedicated to RP2040 effect commands.

Replace Motor FeatherWing pump control with direct RP2040 GP8 MOSFET drive while keeping GP7 assigned to the FP-S14B claw servo.

Update both firmware sketches and DeviceConfig headers to match the revised controller responsibilities, serial command flow, and output mappings.

Restructure the KiCad project by removing the legacy NeoPXL8 and motor-and-claw sheets, adding the new core-strip and pump-and-claw sheets, and aligning the block hierarchy and power sheet with the current 5V bus plus 3V filament rail model.

Synchronize README, ASCII wiring, Mermaid wiring, Fritzing mapping, wire labels, KiCad netmaps, and BOM so the documented hardware revision matches the firmware and schematics.

Standardize beam and filament resistor values across the documentation and KiCad sources and retain a compatibility copy of the older KiCad netmap without leaving contradictory power-rail guidance.
Parts:
- R701, R702, R703: value 1R -> 10R
Changed lines of the file:
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@@
   (title_block
     (title "Beam RGB and Peltier")
-    (date "2026-03-30")
-    (rev "B")
+    (date "2026-03-31")
+    (rev "C")
   )
   (hierarchical_label "BEAM_R_PWM" (shape input) (at 20 90 180)
@@
     (effects (font (size 1.27 1.27)) (justify right))
   )
-  (hierarchical_label "+12V_MAIN" (shape input) (at 20 112 180)
+  (hierarchical_label "+5V_BUS" (shape input) (at 20 112 180)
     (effects (font (size 1.27 1.27)) (justify right))
   )
@@
     (in_bom yes) (on_board yes)
     (property "Reference" "R701" (id 0) (at 74 89.65 0))
-    (property "Value" "1R" (id 1) (at 74 94.73 0))
+    (property "Value" "10R" (id 1) (at 74 94.73 0))
     (property "Footprint" "Resistor_SMD:R_0805_2012Metric" (id 2) (at 74 92.19 0)
       (effects (font (size 1.27 1.27)) hide)
@@
     (in_bom yes) (on_board yes)
     (property "Reference" "R702" (id 0) (at 74 92.19 0))
-    (property "Value" "1R" (id 1) (at 74 97.27 0))
+    (property "Value" "10R" (id 1) (at 74 97.27 0))
     (property "Footprint" "Resistor_SMD:R_0805_2012Metric" (id 2) (at 74 94.73 0)
       (effects (font (size 1.27 1.27)) hide)
@@
     (in_bom yes) (on_board yes)
     (property "Reference" "R703" (id 0) (at 74 94.73 0))
-    (property "Value" "1R" (id 1) (at 74 99.81 0))
+    (property "Value" "10R" (id 1) (at 74 99.81 0))
     (property "Footprint" "Resistor_SMD:R_0805_2012Metric" (id 2) (at 74 97.27 0)
       (effects (font (size 1.27 1.27)) hide)
@@
     )
     (path "/0459a7f8-2ca2-4539-b326-d3ceb5aab69f"
-      (reference "R701") (unit 1) (value "1R") (footprint "")
+      (reference "R701") (unit 1) (value "10R") (footprint "")
     )
     (path "/9719f36e-d8f1-4feb-afcf-95f4de9033ce"
-      (reference "R702") (unit 1) (value "1R") (footprint "")
+      (reference "R702") (unit 1) (value "10R") (footprint "")
     )
     (path "/36d20e64-42bc-4b8c-b574-dd32f6ce2f85"
-      (reference "R703") (unit 1) (value "1R") (footprint "")
-    )
-  )
+      (reference "R703") (unit 1) (value "10R") (footprint "")
+    )
+  )

Commit message: Merge Box updates, normalize circuit layout, and add Box sync workflow
Parts:
- removed J703: Peltier_Load_Out, Adafruit_Eagle:JST-PH-2-THM, symbol Connector_Generic:Conn_01x02
- J701: value Beam_PWM_Inputs -> PropMaker_PWM_Inputs
- J702: value RGB_Load_Out -> LED_3_9W_Out
Other:
- note added: "Prop-Maker LED output stage 3 control channels from RP2040 4th pin on output connector carries +5V bus for the LED load"
- title: Beam RGB and Peltier -> Prop-Maker LED Outputs
Changed lines of the file:
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@@
   (paper "A4")
   (title_block
-    (title "Beam RGB and Peltier")
-    (date "2026-03-31")
-    (rev "C")
+    (title "Prop-Maker LED Outputs")
+    (date "2026-04-08")
+    (rev "D")
   )
-  (hierarchical_label "BEAM_R_PWM" (shape input) (at 20 90 180)
+  (hierarchical_label "PROP_LED1_PWM" (shape input) (at 20 90 180)
     (effects (font (size 1.27 1.27)) (justify right))
   )
-  (hierarchical_label "BEAM_G_PWM" (shape input) (at 20 94 180)
+  (hierarchical_label "PROP_LED2_PWM" (shape input) (at 20 94 180)
     (effects (font (size 1.27 1.27)) (justify right))
   )
-  (hierarchical_label "BEAM_B_PWM" (shape input) (at 20 98 180)
+  (hierarchical_label "PROP_LED3_PWM" (shape input) (at 20 98 180)
     (effects (font (size 1.27 1.27)) (justify right))
   )
-  (hierarchical_label "PELTIER_EN" (shape input) (at 20 102 180)
+  (hierarchical_label "+5V_BUS" (shape input) (at 20 102 180)
     (effects (font (size 1.27 1.27)) (justify right))
   )
-  (hierarchical_label "+5V_BUS" (shape input) (at 20 112 180)
-    (effects (font (size 1.27 1.27)) (justify right))
-  )
-  (hierarchical_label "GND_COMMON" (shape input) (at 20 116 180)
+  (hierarchical_label "GND_COMMON" (shape input) (at 20 106 180)
     (effects (font (size 1.27 1.27)) (justify right))
   )
@@
     (in_bom yes) (on_board yes)
     (property "Reference" "J701" (id 0) (at 60 89 0))
-    (property "Value" "Beam_PWM_Inputs" (id 1) (at 62.54 96 90))
+    (property "Value" "PropMaker_PWM_Inputs" (id 1) (at 62.54 96 90))
     (property "Footprint" "Adafruit_Eagle:1X04-BIG" (id 2) (at 60 96 0)
       (effects (font (size 1.27 1.27)) hide)
@@
     (in_bom yes) (on_board yes)
     (property "Reference" "J702" (id 0) (at 88 89 0))
-    (property "Value" "RGB_Load_Out" (id 1) (at 90.54 96 90))
+    (property "Value" "LED_3_9W_Out" (id 1) (at 90.54 96 90))
     (property "Footprint" "Adafruit_Eagle:1X04-3.5MM" (id 2) (at 88 96 0)
       (effects (font (size 1.27 1.27)) hide)
@@
     (pin "3")
     (pin "4")
-  )
-  (symbol (lib_id "Connector_Generic:Conn_01x02") (at 106 108 0) (unit 1)
-    (in_bom yes) (on_board yes)
-    (property "Reference" "J703" (id 0) (at 106 103 0))
-    (property "Value" "Peltier_Load_Out" (id 1) (at 108.54 108 90))
-    (property "Footprint" "Adafruit_Eagle:JST-PH-2-THM" (id 2) (at 106 108 0)
-      (effects (font (size 1.27 1.27)) hide)
-    )
-    (property "Datasheet" "" (id 3) (at 106 108 0))
-    (pin "1")
-    (pin "2")
   )
   (symbol (lib_id "Device:R") (at 74 92.19 0) (unit 1)
@@
     (pin "2")
   )
-  (label "BEAM_R_PWM" (at 54.92 92.19 0)
+  (label "PROP_LED1_PWM" (at 54.92 92.19 0)
     (effects (font (size 1.27 1.27)) (justify left bottom))
   )
-  (label "BEAM_G_PWM" (at 54.92 94.73 0)
+  (label "PROP_LED2_PWM" (at 54.92 94.73 0)
     (effects (font (size 1.27 1.27)) (justify left bottom))
   )
-  (label "BEAM_B_PWM" (at 54.92 97.27 0)
+  (label "PROP_LED3_PWM" (at 54.92 97.27 0)
     (effects (font (size 1.27 1.27)) (justify left bottom))
   )
-  (label "PELTIER_EN" (at 54.92 99.81 0)
+  (label "GND_COMMON" (at 54.92 99.81 0)
     (effects (font (size 1.27 1.27)) (justify left bottom))
   )
-  (label "GND_COMMON" (at 82.92 99.81 0)
+  (label "+5V_BUS" (at 82.92 99.81 0)
     (effects (font (size 1.27 1.27)) (justify left bottom))
   )
-  (label "PELTIER_EN" (at 100.92 106.73 0)
-    (effects (font (size 1.27 1.27)) (justify left bottom))
-  )
-  (label "GND_COMMON" (at 100.92 109.27 0)
-    (effects (font (size 1.27 1.27)) (justify left bottom))
+  (text "Prop-Maker LED output stage\n3 control channels from RP2040\n4th pin on output connector carries +5V bus for the LED load" (at 60 84 0)
+    (effects (font (size 1.27 1.27)) (justify left top))
   )
   (wire (pts (xy 20 90) (xy 24 90))
@@
     (stroke (width 0) (type default))
   )
-  (wire (pts (xy 20 112) (xy 24 112))
-    (stroke (width 0) (type default))
-  )
-  (wire (pts (xy 20 116) (xy 24 116))
+  (wire (pts (xy 20 106) (xy 24 106))
     (stroke (width 0) (type default))
   )
@@
     (stroke (width 0) (type default))
   )
-  (wire (pts (xy 100.92 106.73) (xy 106 106.73))
-    (stroke (width 0) (type default))
-  )
-  (wire (pts (xy 100.92 109.27) (xy 106 109.27))
-    (stroke (width 0) (type default))
-  )
   (sheet_instances
     (path "/" (page "7"))
@@
   (symbol_instances
     (path "/c6f95c19-e7b5-4e42-a3da-2cf6df70e274"
-      (reference "J701") (unit 1) (value "Beam_PWM_Inputs") (footprint "Adafruit_Eagle:1X04-BIG")
+      (reference "J701") (unit 1) (value "PropMaker_PWM_Inputs") (footprint "Adafruit_Eagle:1X04-BIG")
     )
     (path "/2c16f2f6-4287-4ab7-b6da-966f2ff65489"
-      (reference "J702") (unit 1) (value "RGB_Load_Out") (footprint "Adafruit_Eagle:1X04-3.5MM")
-    )
-    (path "/5e21f623-60cf-47af-af40-1bd523f5ce16"
-      (reference "J703") (unit 1) (value "Peltier_Load_Out") (footprint "Adafruit_Eagle:JST-PH-2-THM")
+      (reference "J702") (unit 1) (value "LED_3_9W_Out") (footprint "Adafruit_Eagle:1X04-3.5MM")
     )
     (path "/0459a7f8-2ca2-4539-b326-d3ceb5aab69f"
