File: circuit/kicad/sheet_filaments.kicad_sch (KiCad schematic)
At the start: 3 parts, among them J601 Filament_PWM_Bus, J602 Filament_Power_In, J603 Filament_Loads_Out

Commit message: Refactor controller roles and update power/resistor schematics
Parts:
- added R601, R602, R603, R604, R605: 10R, symbol Device:R
Changed lines of the file:
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@@
     (pin "5")
+  )
+  (symbol (lib_id "Device:R") (at 96 90.92 0) (unit 1)
+    (in_bom yes) (on_board yes)
+    (property "Reference" "R601" (id 0) (at 96 88.38 0))
+    (property "Value" "10R" (id 1) (at 96 93.46 0))
+    (property "Footprint" "" (id 2) (at 96 90.92 0)
+      (effects (font (size 1.27 1.27)) hide)
+    )
+    (property "Datasheet" "" (id 3) (at 96 90.92 0)
+      (effects (font (size 1.27 1.27)) hide)
+    )
+    (pin "1")
+    (pin "2")
+  )
+  (symbol (lib_id "Device:R") (at 96 93.46 0) (unit 1)
+    (in_bom yes) (on_board yes)
+    (property "Reference" "R602" (id 0) (at 96 90.92 0))
+    (property "Value" "10R" (id 1) (at 96 96 0))
+    (property "Footprint" "" (id 2) (at 96 93.46 0)
+      (effects (font (size 1.27 1.27)) hide)
+    )
+    (property "Datasheet" "" (id 3) (at 96 93.46 0)
+      (effects (font (size 1.27 1.27)) hide)
+    )
+    (pin "1")
+    (pin "2")
+  )
+  (symbol (lib_id "Device:R") (at 96 96 0) (unit 1)
+    (in_bom yes) (on_board yes)
+    (property "Reference" "R603" (id 0) (at 96 93.46 0))
+    (property "Value" "10R" (id 1) (at 96 98.54 0))
+    (property "Footprint" "" (id 2) (at 96 96 0)
+      (effects (font (size 1.27 1.27)) hide)
+    )
+    (property "Datasheet" "" (id 3) (at 96 96 0)
+      (effects (font (size 1.27 1.27)) hide)
+    )
+    (pin "1")
+    (pin "2")
+  )
+  (symbol (lib_id "Device:R") (at 96 98.54 0) (unit 1)
+    (in_bom yes) (on_board yes)
+    (property "Reference" "R604" (id 0) (at 96 96 0))
+    (property "Value" "10R" (id 1) (at 96 101.08 0))
+    (property "Footprint" "" (id 2) (at 96 98.54 0)
+      (effects (font (size 1.27 1.27)) hide)
+    )
+    (property "Datasheet" "" (id 3) (at 96 98.54 0)
+      (effects (font (size 1.27 1.27)) hide)
+    )
+    (pin "1")
+    (pin "2")
+  )
+  (symbol (lib_id "Device:R") (at 96 101.08 0) (unit 1)
+    (in_bom yes) (on_board yes)
+    (property "Reference" "R605" (id 0) (at 96 98.54 0))
+    (property "Value" "10R" (id 1) (at 96 103.62 0))
+    (property "Footprint" "" (id 2) (at 96 101.08 0)
+      (effects (font (size 1.27 1.27)) hide)
+    )
+    (property "Datasheet" "" (id 3) (at 96 101.08 0)
+      (effects (font (size 1.27 1.27)) hide)
+    )
+    (pin "1")
+    (pin "2")
   )
   (label "SPARK1_PWM" (at 56.92 89.65 0)
@@
       (reference "J603") (unit 1) (value "Filament_Loads_Out") (footprint "Adafruit_Eagle:1X06")
     )
+    (path "/71f4a326-69be-47b7-98bb-2f9aee56e53e"
+      (reference "R601") (unit 1) (value "10R") (footprint "")
+    )
+    (path "/d4b15f95-a0d4-4528-a807-ee1159ca568e"
+      (reference "R602") (unit 1) (value "10R") (footprint "")
+    )
+    (path "/d4931538-22d8-47f6-bcee-58f67e1783b7"
+      (reference "R603") (unit 1) (value "10R") (footprint "")
+    )
+    (path "/a72f966c-7ebd-4599-90bc-3e300eb97cf4"
+      (reference "R604") (unit 1) (value "10R") (footprint "")
+    )
+    (path "/d31de17e-e251-4fd2-ab41-1ff29dcf76e5"
+      (reference "R605") (unit 1) (value "10R") (footprint "")
+    )
   )
