File: circuit/kicad/sheet_filaments.kicad_sch (KiCad schematic)
At the start: 8 parts, among them J601 Filament_PWM_Bus, J602 Filament_Power_In, J603 Filament_Loads_Out

Commit message: Assign standard SMD footprints to resistors and fuses
Parts:
- R601, R602, R603, R604, R605: footprint (none) -> Resistor_SMD:R_0805_2012Metric
Changed lines of the file:
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@@
     (property "Reference" "R601" (id 0) (at 96 87.11 0))
     (property "Value" "10R" (id 1) (at 96 92.19 0))
-    (property "Footprint" "" (id 2) (at 96 89.65 0)
+    (property "Footprint" "Resistor_SMD:R_0805_2012Metric" (id 2) (at 96 89.65 0)
       (effects (font (size 1.27 1.27)) hide)
     )
@@
     (property "Reference" "R602" (id 0) (at 96 89.65 0))
     (property "Value" "10R" (id 1) (at 96 94.73 0))
-    (property "Footprint" "" (id 2) (at 96 92.19 0)
+    (property "Footprint" "Resistor_SMD:R_0805_2012Metric" (id 2) (at 96 92.19 0)
       (effects (font (size 1.27 1.27)) hide)
     )
@@
     (property "Reference" "R603" (id 0) (at 96 92.19 0))
     (property "Value" "10R" (id 1) (at 96 97.27 0))
-    (property "Footprint" "" (id 2) (at 96 94.73 0)
+    (property "Footprint" "Resistor_SMD:R_0805_2012Metric" (id 2) (at 96 94.73 0)
       (effects (font (size 1.27 1.27)) hide)
     )
@@
     (property "Reference" "R604" (id 0) (at 96 94.73 0))
     (property "Value" "10R" (id 1) (at 96 99.81 0))
-    (property "Footprint" "" (id 2) (at 96 97.27 0)
+    (property "Footprint" "Resistor_SMD:R_0805_2012Metric" (id 2) (at 96 97.27 0)
       (effects (font (size 1.27 1.27)) hide)
     )
@@
     (property "Reference" "R605" (id 0) (at 96 97.27 0))
     (property "Value" "10R" (id 1) (at 96 102.35 0))
-    (property "Footprint" "" (id 2) (at 96 99.81 0)
+    (property "Footprint" "Resistor_SMD:R_0805_2012Metric" (id 2) (at 96 99.81 0)
       (effects (font (size 1.27 1.27)) hide)
     )

Commit message: Migrate Orciny device to single-strip core and GPIO pump control
Replace the M0 NeoPXL8-based core controller with a single 30-pixel NeoPixel strip on D13 and keep Serial1 TX dedicated to RP2040 effect commands.

Replace Motor FeatherWing pump control with direct RP2040 GP8 MOSFET drive while keeping GP7 assigned to the FP-S14B claw servo.

Update both firmware sketches and DeviceConfig headers to match the revised controller responsibilities, serial command flow, and output mappings.

Restructure the KiCad project by removing the legacy NeoPXL8 and motor-and-claw sheets, adding the new core-strip and pump-and-claw sheets, and aligning the block hierarchy and power sheet with the current 5V bus plus 3V filament rail model.

Synchronize README, ASCII wiring, Mermaid wiring, Fritzing mapping, wire labels, KiCad netmaps, and BOM so the documented hardware revision matches the firmware and schematics.

Standardize beam and filament resistor values across the documentation and KiCad sources and retain a compatibility copy of the older KiCad netmap without leaving contradictory power-rail guidance.
Changed lines of the file:
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@@
   (title_block
     (title "Spark and Pulse Filaments")
-    (date "2026-03-30")
-    (rev "B")
+    (date "2026-03-31")
+    (rev "C")
   )
   (hierarchical_label "SPARK1_PWM" (shape input) (at 20 90 180)
@@
     (effects (font (size 1.27 1.27)) (justify right))
   )
-  (hierarchical_label "+12V_MAIN" (shape input) (at 20 112 180)
+  (hierarchical_label "+3V_FILAMENT" (shape input) (at 20 112 180)
     (effects (font (size 1.27 1.27)) (justify right))
   )
@@
     (effects (font (size 1.27 1.27)) (justify left bottom))
   )
-  (label "+12V_MAIN" (at 84.92 106.73 0)
+  (label "+3V_FILAMENT" (at 84.92 106.73 0)
     (effects (font (size 1.27 1.27)) (justify left bottom))
   )

Commit message: updated paperwork
Parts:
- removed R605: 10R, Resistor_SMD:R_0805_2012Metric, symbol Device:R
- J601: footprint Adafruit_Eagle:1X06 -> Adafruit_Eagle:1X05; symbol Connector_Generic:Conn_01x06 -> Connector_Generic:Conn_01x05
- J603: footprint Adafruit_Eagle:1X06 -> Adafruit_Eagle:1X04-BIG; symbol Connector_Generic:Conn_01x05 -> Connector_Generic:Conn_01x04
Other:
- title: Spark and Pulse Filaments -> Spark Filaments
Changed lines of the file:
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@@
   (paper "A4")
   (title_block
-    (title "Spark and Pulse Filaments")
+    (title "Spark Filaments")
     (date "2026-03-31")
     (rev "C")
@@
     (effects (font (size 1.27 1.27)) (justify right))
   )
-  (hierarchical_label "PULSE_PWM" (shape input) (at 20 106 180)
-    (effects (font (size 1.27 1.27)) (justify right))
-  )
   (hierarchical_label "+3V_FILAMENT" (shape input) (at 20 112 180)
     (effects (font (size 1.27 1.27)) (justify right))
@@
     (effects (font (size 1.27 1.27)) (justify right))
   )
-  (symbol (lib_id "Connector_Generic:Conn_01x06") (at 62 96 0) (unit 1)
+  (symbol (lib_id "Connector_Generic:Conn_01x05") (at 62 96 0) (unit 1)
     (in_bom yes) (on_board yes)
     (property "Reference" "J601" (id 0) (at 62 88 0))
     (property "Value" "Filament_PWM_Bus" (id 1) (at 64.54 96 90))
-    (property "Footprint" "Adafruit_Eagle:1X06" (id 2) (at 62 96 0)
+    (property "Footprint" "Adafruit_Eagle:1X05" (id 2) (at 62 96 0)
       (effects (font (size 1.27 1.27)) hide)
     )
@@
     (pin "4")
     (pin "5")
-    (pin "6")
   )
   (symbol (lib_id "Connector_Generic:Conn_01x02") (at 90 108 0) (unit 1)
@@
     (pin "2")
   )
-  (symbol (lib_id "Connector_Generic:Conn_01x05") (at 106 96 0) (unit 1)
+  (symbol (lib_id "Connector_Generic:Conn_01x04") (at 106 94.73 0) (unit 1)
     (in_bom yes) (on_board yes)
     (property "Reference" "J603" (id 0) (at 106 89 0))
-    (property "Value" "Filament_Loads_Out" (id 1) (at 108.54 96 90))
-    (property "Footprint" "Adafruit_Eagle:1X06" (id 2) (at 106 96 0)
-      (effects (font (size 1.27 1.27)) hide)
-    )
-    (property "Datasheet" "" (id 3) (at 106 96 0))
+    (property "Value" "Filament_Loads_Out" (id 1) (at 108.54 94.73 90))
+    (property "Footprint" "Adafruit_Eagle:1X04-BIG" (id 2) (at 106 94.73 0)
+      (effects (font (size 1.27 1.27)) hide)
+    )
+    (property "Datasheet" "" (id 3) (at 106 94.73 0))
     (pin "1")
     (pin "2")
     (pin "3")
     (pin "4")
-    (pin "5")
   )
   (symbol (lib_id "Device:R") (at 96 89.65 0) (unit 1)
@@
     (pin "2")
   )
-  (symbol (lib_id "Device:R") (at 96 99.81 0) (unit 1)
-    (in_bom yes) (on_board yes)
-    (property "Reference" "R605" (id 0) (at 96 97.27 0))
-    (property "Value" "10R" (id 1) (at 96 102.35 0))
-    (property "Footprint" "Resistor_SMD:R_0805_2012Metric" (id 2) (at 96 99.81 0)
-      (effects (font (size 1.27 1.27)) hide)
-    )
-    (property "Datasheet" "" (id 3) (at 96 99.81 0)
-      (effects (font (size 1.27 1.27)) hide)
-    )
-    (pin "1")
-    (pin "2")
-  )
   (label "SPARK1_PWM" (at 56.92 89.65 0)
     (effects (font (size 1.27 1.27)) (justify left bottom))
@@
     (effects (font (size 1.27 1.27)) (justify left bottom))
   )
-  (label "PULSE_PWM" (at 56.92 99.81 0)
-    (effects (font (size 1.27 1.27)) (justify left bottom))
-  )
-  (label "GND_COMMON" (at 56.92 102.35 0)
+  (label "GND_COMMON" (at 56.92 99.81 0)
     (effects (font (size 1.27 1.27)) (justify left bottom))
   )
@@
     (stroke (width 0) (type default))
   )
-  (wire (pts (xy 20 106) (xy 24 106))
-    (stroke (width 0) (type default))
-  )
   (wire (pts (xy 20 112) (xy 24 112))
     (stroke (width 0) (type default))
@@
     (stroke (width 0) (type default))
   )
-  (wire (pts (xy 56.92 102.35) (xy 62 102.35))
-    (stroke (width 0) (type default))
-  )
   (wire (pts (xy 84.92 106.73) (xy 90 106.73))
     (stroke (width 0) (type default))
@@
   )
   (wire (pts (xy 100.92 98.54) (xy 106 98.54))
-    (stroke (width 0) (type default))
-  )
-  (wire (pts (xy 62 99.81) (xy 94.73 99.81))
-    (stroke (width 0) (type default))
-  )
-  (wire (pts (xy 97.27 99.81) (xy 100.92 99.81))
-    (stroke (width 0) (type default))
-  )
-  (wire (pts (xy 100.92 99.81) (xy 100.92 101.08))
-    (stroke (width 0) (type default))
-  )
-  (wire (pts (xy 100.92 101.08) (xy 106 101.08))
     (stroke (width 0) (type default))
   )
@@
   (symbol_instances
     (path "/2f21026e-9ee1-4057-8ec8-8d3ef0e48997"
-      (reference "J601") (unit 1) (value "Filament_PWM_Bus") (footprint "Adafruit_Eagle:1X06")
+      (reference "J601") (unit 1) (value "Filament_PWM_Bus") (footprint "Adafruit_Eagle:1X05")
     )
     (path "/66cc5860-8fac-4515-9657-c71f6f32aad1"
@@
     )
     (path "/6254f9f4-9be4-4bc3-9f0a-2cae6f173013"
-      (reference "J603") (unit 1) (value "Filament_Loads_Out") (footprint "Adafruit_Eagle:1X06")
+      (reference "J603") (unit 1) (value "Filament_Loads_Out") (footprint "Adafruit_Eagle:1X04-BIG")
     )
     (path "/71f4a326-69be-47b7-98bb-2f9aee56e53e"
@@
       (reference "R604") (unit 1) (value "10R") (footprint "")
     )
-    (path "/d31de17e-e251-4fd2-ab41-1ff29dcf76e5"
-      (reference "R605") (unit 1) (value "10R") (footprint "")
-    )
-  )
+  )
