File: circuit/kicad/sheet_filaments.kicad_sch (KiCad schematic)
At the start: 8 parts, among them J601 Filament_PWM_Bus, J602 Filament_Power_In, J603 Filament_Loads_Out

Commit message: Merge Box updates, normalize circuit layout, and add Box sync workflow
Parts:
- removed R605: 10R, Resistor_SMD:R_0805_2012Metric, symbol Device:R
- J?: renamed from J601; footprint Adafruit_Eagle:1X06 -> Adafruit_Eagle:1X05; symbol Connector_Generic:Conn_01x06 -> Connector_Generic:Conn_01x05
- J?: renamed from J603; footprint Adafruit_Eagle:1X06 -> Adafruit_Eagle:1X04-BIG; symbol Connector_Generic:Conn_01x05 -> Connector_Generic:Conn_01x04
- renumbered J602 to J?, R601 to R?, R604 to R?, R603 to R?, R602 to R?
Other:
- title: Spark and Pulse Filaments -> Spark Filaments
