File: circuit/kicad/sheet_power.kicad_sch (KiCad schematic)
At the start: 2 parts, among them J801 Main_12V_In, J802 Power_Distribution

Commit message: Refactor controller roles and update power/resistor schematics
Parts:
- added F801: Fuse_5V_Logic, symbol Device:Fuse
- added F802: Fuse_12V_Branch, symbol Device:Fuse
- added F803: Fuse_5V_Act, symbol Device:Fuse
- J802: footprint Adafruit_Eagle:1X03 -> Adafruit_Eagle:1X04; symbol Connector_Generic:Conn_01x03 -> Connector_Generic:Conn_01x04
Changed lines of the file:
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@@
+    (effects (font (size 1.27 1.27)) (justify left))
+  )
+  (hierarchical_label "+5V_ACT" (shape output) (at 120 164 0)
     (effects (font (size 1.27 1.27)) (justify left))
   )
@@
     (pin "2")
   )
-  (symbol (lib_id "Connector_Generic:Conn_01x03") (at 90 152 0) (unit 1)
+  (symbol (lib_id "Connector_Generic:Conn_01x04") (at 90 152 0) (unit 1)
     (in_bom yes) (on_board yes)
     (property "Reference" "J802" (id 0) (at 90 146 0))
     (property "Value" "Power_Distribution" (id 1) (at 92.54 152 90))
-    (property "Footprint" "Adafruit_Eagle:1X03" (id 2) (at 90 152 0)
+    (property "Footprint" "Adafruit_Eagle:1X04" (id 2) (at 90 152 0)
       (effects (font (size 1.27 1.27)) hide)
     )
@@
     (pin "2")
     (pin "3")
+    (pin "4")
+  )
+  (symbol (lib_id "Device:Fuse") (at 74 146 0) (unit 1)
+    (in_bom yes) (on_board yes)
+    (property "Reference" "F801" (id 0) (at 74 143.46 0))
+    (property "Value" "Fuse_5V_Logic" (id 1) (at 74 148.54 0))
+    (property "Footprint" "" (id 2) (at 74 146 0)
+      (effects (font (size 1.27 1.27)) hide)
+    )
+    (property "Datasheet" "" (id 3) (at 74 146 0)
+      (effects (font (size 1.27 1.27)) hide)
+    )
+    (pin "1")
+    (pin "2")
+  )
+  (symbol (lib_id "Device:Fuse") (at 74 152 0) (unit 1)
+    (in_bom yes) (on_board yes)
+    (property "Reference" "F802" (id 0) (at 74 149.46 0))
+    (property "Value" "Fuse_12V_Branch" (id 1) (at 74 154.54 0))
+    (property "Footprint" "" (id 2) (at 74 152 0)
+      (effects (font (size 1.27 1.27)) hide)
+    )
+    (property "Datasheet" "" (id 3) (at 74 152 0)
+      (effects (font (size 1.27 1.27)) hide)
+    )
+    (pin "1")
+    (pin "2")
+  )
+  (symbol (lib_id "Device:Fuse") (at 74 158 0) (unit 1)
+    (in_bom yes) (on_board yes)
+    (property "Reference" "F803" (id 0) (at 74 155.46 0))
+    (property "Value" "Fuse_5V_Act" (id 1) (at 74 160.54 0))
+    (property "Footprint" "" (id 2) (at 74 158 0)
+      (effects (font (size 1.27 1.27)) hide)
+    )
+    (property "Datasheet" "" (id 3) (at 74 158 0)
+      (effects (font (size 1.27 1.27)) hide)
+    )
+    (pin "1")
+    (pin "2")
   )
   (label "+12V_MAIN" (at 56.92 150.73 0)
@@
     (effects (font (size 1.27 1.27)) (justify left bottom))
   )
+  (label "+5V_ACT" (at 84.92 157.08 0)
+    (effects (font (size 1.27 1.27)) (justify left bottom))
+  )
   (wire (pts (xy 120 146) (xy 116 146))
     (stroke (width 0) (type default))
@@
   )
   (wire (pts (xy 120 158) (xy 116 158))
+    (stroke (width 0) (type default))
+  )
+  (wire (pts (xy 120 164) (xy 116 164))
     (stroke (width 0) (type default))
   )
@@
     (stroke (width 0) (type default))
   )
+  (wire (pts (xy 84.92 157.08) (xy 90 157.08))
+    (stroke (width 0) (type default))
+  )
   (sheet_instances
     (path "/" (page "8"))
@@
     )
     (path "/72029b2f-7ef0-4522-9237-4f66125c3afd"
-      (reference "J802") (unit 1) (value "Power_Distribution") (footprint "Adafruit_Eagle:1X03")
+      (reference "J802") (unit 1) (value "Power_Distribution") (footprint "Adafruit_Eagle:1X04")
+    )
+    (path "/03c2f827-baf7-4f09-9f67-39ddb07f8129"
+      (reference "F801") (unit 1) (value "Fuse_5V_Logic") (footprint "")
+    )
+    (path "/9b25e1e7-ec6f-433b-92f5-4bffb93a2ea2"
+      (reference "F802") (unit 1) (value "Fuse_12V_Branch") (footprint "")
+    )
+    (path "/7d4eccf9-aeb2-44b3-bc24-e6bbabf67667"
+      (reference "F803") (unit 1) (value "Fuse_5V_Act") (footprint "")
     )
   )
