File: circuit/kicad/sheet_power.kicad_sch (KiCad schematic)
At the start: 5 parts, among them J801 Main_12V_In, J802 Power_Distribution

Commit message: Assign standard SMD footprints to resistors and fuses
Parts:
- F801, F802, F803: footprint (none) -> Fuse:Fuse_1206_3216Metric
Changed lines of the file:
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@@
     (property "Reference" "F801" (id 0) (at 74 146.92 0))
     (property "Value" "Fuse_5V_Logic" (id 1) (at 74 152 0))
-    (property "Footprint" "" (id 2) (at 74 149.46 0)
+    (property "Footprint" "Fuse:Fuse_1206_3216Metric" (id 2) (at 74 149.46 0)
       (effects (font (size 1.27 1.27)) hide)
     )
@@
     (property "Reference" "F802" (id 0) (at 74 149.46 0))
     (property "Value" "Fuse_12V_Branch" (id 1) (at 74 154.54 0))
-    (property "Footprint" "" (id 2) (at 74 152 0)
+    (property "Footprint" "Fuse:Fuse_1206_3216Metric" (id 2) (at 74 152 0)
       (effects (font (size 1.27 1.27)) hide)
     )
@@
     (property "Reference" "F803" (id 0) (at 74 154.54 0))
     (property "Value" "Fuse_5V_Act" (id 1) (at 74 159.62 0))
-    (property "Footprint" "" (id 2) (at 74 157.08 0)
+    (property "Footprint" "Fuse:Fuse_1206_3216Metric" (id 2) (at 74 157.08 0)
       (effects (font (size 1.27 1.27)) hide)
     )

Commit message: Migrate Orciny device to single-strip core and GPIO pump control
Replace the M0 NeoPXL8-based core controller with a single 30-pixel NeoPixel strip on D13 and keep Serial1 TX dedicated to RP2040 effect commands.

Replace Motor FeatherWing pump control with direct RP2040 GP8 MOSFET drive while keeping GP7 assigned to the FP-S14B claw servo.

Update both firmware sketches and DeviceConfig headers to match the revised controller responsibilities, serial command flow, and output mappings.

Restructure the KiCad project by removing the legacy NeoPXL8 and motor-and-claw sheets, adding the new core-strip and pump-and-claw sheets, and aligning the block hierarchy and power sheet with the current 5V bus plus 3V filament rail model.

Synchronize README, ASCII wiring, Mermaid wiring, Fritzing mapping, wire labels, KiCad netmaps, and BOM so the documented hardware revision matches the firmware and schematics.

Standardize beam and filament resistor values across the documentation and KiCad sources and retain a compatibility copy of the older KiCad netmap without leaving contradictory power-rail guidance.
Parts:
- removed F803: Fuse_5V_Act, Fuse:Fuse_1206_3216Metric, symbol Device:Fuse
- F801: value Fuse_5V_Logic -> Fuse_5V_Bus
- F802: value Fuse_12V_Branch -> Fuse_3V_Filament
- J801: value Main_12V_In -> Main_5V_In
- J802: footprint Adafruit_Eagle:1X04 -> Adafruit_Eagle:1X03; symbol Connector_Generic:Conn_01x04 -> Connector_Generic:Conn_01x03
Changed lines of the file:
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@@
   (title_block
     (title "Power Domains")
-    (date "2026-03-30")
-    (rev "B")
+    (date "2026-03-31")
+    (rev "C")
   )
-  (hierarchical_label "+5V_LOGIC" (shape output) (at 120 146 0)
+  (hierarchical_label "+5V_BUS" (shape output) (at 120 146 0)
     (effects (font (size 1.27 1.27)) (justify left))
   )
-  (hierarchical_label "+12V_MAIN" (shape output) (at 120 152 0)
+  (hierarchical_label "+3V_FILAMENT" (shape output) (at 120 152 0)
     (effects (font (size 1.27 1.27)) (justify left))
   )
@@
     (effects (font (size 1.27 1.27)) (justify left))
   )
-  (hierarchical_label "+5V_ACT" (shape output) (at 120 164 0)
-    (effects (font (size 1.27 1.27)) (justify left))
-  )
   (symbol (lib_id "Connector_Generic:Conn_01x02") (at 62 152 0) (unit 1)
     (in_bom yes) (on_board yes)
     (property "Reference" "J801" (id 0) (at 62 147 0))
-    (property "Value" "Main_12V_In" (id 1) (at 64.54 152 90))
+    (property "Value" "Main_5V_In" (id 1) (at 64.54 152 90))
     (property "Footprint" "Adafruit_Eagle:DCJACK_2MM_PTH" (id 2) (at 62 152 0)
       (effects (font (size 1.27 1.27)) hide)
@@
     (pin "2")
   )
-  (symbol (lib_id "Connector_Generic:Conn_01x04") (at 90 152 0) (unit 1)
+  (symbol (lib_id "Connector_Generic:Conn_01x03") (at 90 152 0) (unit 1)
     (in_bom yes) (on_board yes)
     (property "Reference" "J802" (id 0) (at 90 146 0))
     (property "Value" "Power_Distribution" (id 1) (at 92.54 152 90))
-    (property "Footprint" "Adafruit_Eagle:1X04" (id 2) (at 90 152 0)
+    (property "Footprint" "Adafruit_Eagle:1X03" (id 2) (at 90 152 0)
       (effects (font (size 1.27 1.27)) hide)
     )
@@
     (pin "2")
     (pin "3")
-    (pin "4")
   )
   (symbol (lib_id "Device:Fuse") (at 74 149.46 0) (unit 1)
     (in_bom yes) (on_board yes)
     (property "Reference" "F801" (id 0) (at 74 146.92 0))
-    (property "Value" "Fuse_5V_Logic" (id 1) (at 74 152 0))
+    (property "Value" "Fuse_5V_Bus" (id 1) (at 74 152 0))
     (property "Footprint" "Fuse:Fuse_1206_3216Metric" (id 2) (at 74 149.46 0)
       (effects (font (size 1.27 1.27)) hide)
@@
     (in_bom yes) (on_board yes)
     (property "Reference" "F802" (id 0) (at 74 149.46 0))
-    (property "Value" "Fuse_12V_Branch" (id 1) (at 74 154.54 0))
+    (property "Value" "Fuse_3V_Filament" (id 1) (at 74 154.54 0))
     (property "Footprint" "Fuse:Fuse_1206_3216Metric" (id 2) (at 74 152 0)
       (effects (font (size 1.27 1.27)) hide)
@@
     (pin "2")
   )
-  (symbol (lib_id "Device:Fuse") (at 74 157.08 0) (unit 1)
-    (in_bom yes) (on_board yes)
-    (property "Reference" "F803" (id 0) (at 74 154.54 0))
-    (property "Value" "Fuse_5V_Act" (id 1) (at 74 159.62 0))
-    (property "Footprint" "Fuse:Fuse_1206_3216Metric" (id 2) (at 74 157.08 0)
-      (effects (font (size 1.27 1.27)) hide)
-    )
-    (property "Datasheet" "" (id 3) (at 74 157.08 0)
-      (effects (font (size 1.27 1.27)) hide)
-    )
-    (pin "1")
-    (pin "2")
-  )
-  (label "+12V_IN" (at 56.92 150.73 0)
+  (label "+5V_IN" (at 56.92 150.73 0)
     (effects (font (size 1.27 1.27)) (justify left bottom))
   )
@@
     (effects (font (size 1.27 1.27)) (justify left bottom))
   )
-  (label "+5V_LOGIC" (at 84.92 149.46 0)
+  (label "+5V_BUS" (at 84.92 149.46 0)
     (effects (font (size 1.27 1.27)) (justify left bottom))
   )
-  (label "+12V_MAIN" (at 84.92 152 0)
+  (label "+3V_FILAMENT" (at 84.92 152 0)
     (effects (font (size 1.27 1.27)) (justify left bottom))
   )
   (label "GND_COMMON" (at 84.92 154.54 0)
-    (effects (font (size 1.27 1.27)) (justify left bottom))
-  )
-  (label "+5V_ACT" (at 84.92 157.08 0)
     (effects (font (size 1.27 1.27)) (justify left bottom))
   )
@@
   )
   (wire (pts (xy 120 158) (xy 116 158))
-    (stroke (width 0) (type default))
-  )
-  (wire (pts (xy 120 164) (xy 116 164))
     (stroke (width 0) (type default))
   )
@@
     (stroke (width 0) (type default))
   )
-  (wire (pts (xy 84.92 157.08) (xy 90 157.08))
-    (stroke (width 0) (type default))
-  )
   (wire (pts (xy 62 150.73) (xy 68 150.73))
     (stroke (width 0) (type default))
   )
-  (wire (pts (xy 68 149.46) (xy 68 157.08))
+  (wire (pts (xy 68 149.46) (xy 68 152))
     (stroke (width 0) (type default))
   )
@@
     (stroke (width 0) (type default))
   )
-  (wire (pts (xy 68 157.08) (xy 72.73 157.08))
-    (stroke (width 0) (type default))
-  )
   (wire (pts (xy 75.27 149.46) (xy 84.92 149.46))
     (stroke (width 0) (type default))
   )
   (wire (pts (xy 75.27 152) (xy 84.92 152))
-    (stroke (width 0) (type default))
-  )
-  (wire (pts (xy 75.27 157.08) (xy 84.92 157.08))
     (stroke (width 0) (type default))
   )
@@
   (symbol_instances
     (path "/aa90f2b9-a98e-4d20-b67e-2b90f7868cc7"
-      (reference "J801") (unit 1) (value "Main_12V_In") (footprint "Adafruit_Eagle:DCJACK_2MM_PTH")
+      (reference "J801") (unit 1) (value "Main_5V_In") (footprint "Adafruit_Eagle:DCJACK_2MM_PTH")
     )
     (path "/72029b2f-7ef0-4522-9237-4f66125c3afd"
-      (reference "J802") (unit 1) (value "Power_Distribution") (footprint "Adafruit_Eagle:1X04")
+      (reference "J802") (unit 1) (value "Power_Distribution") (footprint "Adafruit_Eagle:1X03")
     )
     (path "/03c2f827-baf7-4f09-9f67-39ddb07f8129"
-      (reference "F801") (unit 1) (value "Fuse_5V_Logic") (footprint "")
+      (reference "F801") (unit 1) (value "Fuse_5V_Bus") (footprint "")
     )
     (path "/9b25e1e7-ec6f-433b-92f5-4bffb93a2ea2"
-      (reference "F802") (unit 1) (value "Fuse_12V_Branch") (footprint "")
-    )
-    (path "/7d4eccf9-aeb2-44b3-bc24-e6bbabf67667"
-      (reference "F803") (unit 1) (value "Fuse_5V_Act") (footprint "")
+      (reference "F802") (unit 1) (value "Fuse_3V_Filament") (footprint "")
     )
   )

Commit message: Merge Box updates, normalize circuit layout, and add Box sync workflow
Parts:
- renumbered F801 to F?, F802 to F?, J802 to J?, J801 to J?
