File: circuit/kicad/sheet_rp2040.kicad_sch (KiCad schematic)
At the start: 2 parts, among them U101 Feather_RP2040, U102 Feather_RP2040_B

Commit message: updated paperwork
Changed lines of the file:
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@@
-    (effects (font (size 1.27 1.27)) (justify left))
-  )
-  (hierarchical_label "PULSE_PWM" (shape output) (at 120 60 0)
     (effects (font (size 1.27 1.27)) (justify left))
   )
@@
     (effects (font (size 1.27 1.27)) (justify left bottom))
   )
-  (label "PULSE_PWM" (at 88.92 66 0)
-    (effects (font (size 1.27 1.27)) (justify left bottom))
-  )
   (label "PROP_LED1_PWM" (at 88.92 68.54 0)
     (effects (font (size 1.27 1.27)) (justify left bottom))
@@
   )
   (wire (pts (xy 120 56) (xy 116 56))
-    (stroke (width 0) (type default))
-  )
-  (wire (pts (xy 120 60) (xy 116 60))
     (stroke (width 0) (type default))
   )
@@
     (stroke (width 0) (type default))
   )
-  (wire (pts (xy 88.92 66) (xy 94 66))
-    (stroke (width 0) (type default))
-  )
