File: circuit/kicad/sheet_rp2040.kicad_sch (KiCad schematic)
At the start: 2 parts, among them U101 Feather_RP2040, U102 Feather_RP2040_B

Commit message: Migrate Orciny device to single-strip core and GPIO pump control
Replace the M0 NeoPXL8-based core controller with a single 30-pixel NeoPixel strip on D13 and keep Serial1 TX dedicated to RP2040 effect commands.

Replace Motor FeatherWing pump control with direct RP2040 GP8 MOSFET drive while keeping GP7 assigned to the FP-S14B claw servo.

Update both firmware sketches and DeviceConfig headers to match the revised controller responsibilities, serial command flow, and output mappings.

Restructure the KiCad project by removing the legacy NeoPXL8 and motor-and-claw sheets, adding the new core-strip and pump-and-claw sheets, and aligning the block hierarchy and power sheet with the current 5V bus plus 3V filament rail model.

Synchronize README, ASCII wiring, Mermaid wiring, Fritzing mapping, wire labels, KiCad netmaps, and BOM so the documented hardware revision matches the firmware and schematics.

Standardize beam and filament resistor values across the documentation and KiCad sources and retain a compatibility copy of the older KiCad netmap without leaving contradictory power-rail guidance.
Changed lines of the file:
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@@
     (effects (font (size 1.27 1.27)) (justify right))
   )
-  (hierarchical_label "+5V_LOGIC" (shape input) (at 20 44 180)
+  (hierarchical_label "+5V_BUS" (shape input) (at 20 44 180)
     (effects (font (size 1.27 1.27)) (justify right))
   )
@@
     (effects (font (size 1.27 1.27)) (justify left))
   )
-  (hierarchical_label "I2C_SDA" (shape bidirectional) (at 120 32 0)
+  (hierarchical_label "PUMP_EN" (shape output) (at 120 32 0)
     (effects (font (size 1.27 1.27)) (justify left))
   )
-  (hierarchical_label "I2C_SCL" (shape bidirectional) (at 120 36 0)
+  (hierarchical_label "SERVO_SIG" (shape output) (at 120 36 0)
     (effects (font (size 1.27 1.27)) (justify left))
   )
@@
     (effects (font (size 1.27 1.27)) (justify left bottom))
   )
-  (label "+5V_LOGIC" (at 66.92 43.65 0)
+  (label "+5V_BUS" (at 66.92 43.65 0)
     (effects (font (size 1.27 1.27)) (justify left bottom))
   )
@@
     (effects (font (size 1.27 1.27)) (justify left bottom))
   )
-  (label "I2C_SDA" (at 66.92 51.27 0)
+  (label "PUMP_EN" (at 66.92 51.27 0)
     (effects (font (size 1.27 1.27)) (justify left bottom))
   )
-  (label "I2C_SCL" (at 66.92 53.81 0)
+  (label "SERVO_SIG" (at 66.92 53.81 0)
     (effects (font (size 1.27 1.27)) (justify left bottom))
   )

Commit message: Merge Box updates, normalize circuit layout, and add Box sync workflow
Other:
- note added: "RP2040 FX controller pins match the current FeatherWing-based DeviceConfig.h"
- note removed: "RP2040 main FX controller pins match firmware DeviceConfig.h"
- title: RP2040 Main Controller -> RP2040 FX Controller
Changed lines of the file:
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@@
   (paper "A4")
   (title_block
-    (title "RP2040 Main Controller")
-    (date "2026-03-30")
-    (rev "B")
+    (title "RP2040 FX Controller")
+    (date "2026-04-08")
+    (rev "C")
   )
   (hierarchical_label "SW1_IN" (shape input) (at 20 30 180)
@@
     (effects (font (size 1.27 1.27)) (justify right))
   )
-  (hierarchical_label "SERIAL_LINK" (shape output) (at 120 28 0)
-    (effects (font (size 1.27 1.27)) (justify left))
-  )
-  (hierarchical_label "PUMP_EN" (shape output) (at 120 32 0)
-    (effects (font (size 1.27 1.27)) (justify left))
-  )
-  (hierarchical_label "SERVO_SIG" (shape output) (at 120 36 0)
-    (effects (font (size 1.27 1.27)) (justify left))
-  )
-  (hierarchical_label "SPARK1_PWM" (shape output) (at 120 42 0)
-    (effects (font (size 1.27 1.27)) (justify left))
-  )
-  (hierarchical_label "SPARK2_PWM" (shape output) (at 120 46 0)
-    (effects (font (size 1.27 1.27)) (justify left))
-  )
-  (hierarchical_label "SPARK3_PWM" (shape output) (at 120 50 0)
-    (effects (font (size 1.27 1.27)) (justify left))
-  )
-  (hierarchical_label "SPARK4_PWM" (shape output) (at 120 54 0)
-    (effects (font (size 1.27 1.27)) (justify left))
-  )
-  (hierarchical_label "PULSE_PWM" (shape output) (at 120 58 0)
-    (effects (font (size 1.27 1.27)) (justify left))
-  )
-  (hierarchical_label "BEAM_R_PWM" (shape output) (at 120 62 0)
-    (effects (font (size 1.27 1.27)) (justify left))
-  )
-  (hierarchical_label "BEAM_G_PWM" (shape output) (at 120 66 0)
-    (effects (font (size 1.27 1.27)) (justify left))
-  )
-  (hierarchical_label "BEAM_B_PWM" (shape output) (at 120 70 0)
-    (effects (font (size 1.27 1.27)) (justify left))
-  )
-  (hierarchical_label "PELTIER_EN" (shape output) (at 120 74 0)
-    (effects (font (size 1.27 1.27)) (justify left))
-  )
-  (text "RP2040 main FX controller pins match firmware DeviceConfig.h" (at 20 16 0)
+  (hierarchical_label "CORE_DATA" (shape output) (at 120 28 0)
+    (effects (font (size 1.27 1.27)) (justify left))
+  )
+  (hierarchical_label "PUMP_EN_OPTIONAL" (shape output) (at 120 32 0)
+    (effects (font (size 1.27 1.27)) (justify left))
+  )
+  (hierarchical_label "I2C_SDA_SERVO_WING" (shape output) (at 120 36 0)
+    (effects (font (size 1.27 1.27)) (justify left))
+  )
+  (hierarchical_label "I2C_SCL_SERVO_WING" (shape output) (at 120 40 0)
+    (effects (font (size 1.27 1.27)) (justify left))
+  )
+  (hierarchical_label "SPARK1_PWM" (shape output) (at 120 44 0)
+    (effects (font (size 1.27 1.27)) (justify left))
+  )
+  (hierarchical_label "SPARK2_PWM" (shape output) (at 120 48 0)
+    (effects (font (size 1.27 1.27)) (justify left))
+  )
+  (hierarchical_label "SPARK3_PWM" (shape output) (at 120 52 0)
+    (effects (font (size 1.27 1.27)) (justify left))
+  )
+  (hierarchical_label "SPARK4_PWM" (shape output) (at 120 56 0)
+    (effects (font (size 1.27 1.27)) (justify left))
+  )
+  (hierarchical_label "PROP_LED1_PWM" (shape output) (at 120 64 0)
+    (effects (font (size 1.27 1.27)) (justify left))
+  )
+  (hierarchical_label "PROP_LED2_PWM" (shape output) (at 120 68 0)
+    (effects (font (size 1.27 1.27)) (justify left))
+  )
+  (hierarchical_label "PROP_LED3_PWM" (shape output) (at 120 72 0)
+    (effects (font (size 1.27 1.27)) (justify left))
+  )
+  (text "RP2040 FX controller pins match the current FeatherWing-based DeviceConfig.h" (at 20 16 0)
     (effects (font (size 1.5 1.5)) (justify left bottom))
   )
@@
     (effects (font (size 1.27 1.27)) (justify left bottom))
   )
-  (label "SERIAL_LINK" (at 66.92 48.73 0)
-    (effects (font (size 1.27 1.27)) (justify left bottom))
-  )
-  (label "PUMP_EN" (at 66.92 51.27 0)
-    (effects (font (size 1.27 1.27)) (justify left bottom))
-  )
-  (label "SERVO_SIG" (at 66.92 53.81 0)
-    (effects (font (size 1.27 1.27)) (justify left bottom))
-  )
-  (label "SPARK1_PWM" (at 66.92 56.35 0)
-    (effects (font (size 1.27 1.27)) (justify left bottom))
-  )
-  (label "SPARK2_PWM" (at 66.92 58.89 0)
-    (effects (font (size 1.27 1.27)) (justify left bottom))
-  )
-  (label "SPARK3_PWM" (at 66.92 61.43 0)
-    (effects (font (size 1.27 1.27)) (justify left bottom))
-  )
-  (label "SPARK4_PWM" (at 66.92 63.97 0)
-    (effects (font (size 1.27 1.27)) (justify left bottom))
-  )
-  (label "PULSE_PWM" (at 88.92 63.46 0)
-    (effects (font (size 1.27 1.27)) (justify left bottom))
-  )
-  (label "BEAM_R_PWM" (at 88.92 66 0)
-    (effects (font (size 1.27 1.27)) (justify left bottom))
-  )
-  (label "BEAM_G_PWM" (at 88.92 68.54 0)
-    (effects (font (size 1.27 1.27)) (justify left bottom))
-  )
-  (label "BEAM_B_PWM" (at 88.92 71.08 0)
-    (effects (font (size 1.27 1.27)) (justify left bottom))
-  )
-  (label "PELTIER_EN" (at 88.92 73.62 0)
+  (label "CORE_DATA" (at 66.92 48.73 0)
+    (effects (font (size 1.27 1.27)) (justify left bottom))
+  )
+  (label "PUMP_EN_OPTIONAL" (at 66.92 51.27 0)
+    (effects (font (size 1.27 1.27)) (justify left bottom))
+  )
+  (label "I2C_SDA_SERVO_WING" (at 66.92 53.81 0)
+    (effects (font (size 1.27 1.27)) (justify left bottom))
+  )
+  (label "I2C_SCL_SERVO_WING" (at 66.92 56.35 0)
+    (effects (font (size 1.27 1.27)) (justify left bottom))
+  )
+  (label "SPARK1_PWM" (at 66.92 58.89 0)
+    (effects (font (size 1.27 1.27)) (justify left bottom))
+  )
+  (label "SPARK2_PWM" (at 66.92 61.43 0)
+    (effects (font (size 1.27 1.27)) (justify left bottom))
+  )
+  (label "SPARK3_PWM" (at 66.92 63.97 0)
+    (effects (font (size 1.27 1.27)) (justify left bottom))
+  )
+  (label "SPARK4_PWM" (at 88.92 63.46 0)
+    (effects (font (size 1.27 1.27)) (justify left bottom))
+  )
+  (label "PROP_LED1_PWM" (at 88.92 68.54 0)
+    (effects (font (size 1.27 1.27)) (justify left bottom))
+  )
+  (label "PROP_LED2_PWM" (at 88.92 71.08 0)
+    (effects (font (size 1.27 1.27)) (justify left bottom))
+  )
+  (label "PROP_LED3_PWM" (at 88.92 73.62 0)
     (effects (font (size 1.27 1.27)) (justify left bottom))
   )
@@
     (stroke (width 0) (type default))
   )
-  (wire (pts (xy 120 42) (xy 116 42))
-    (stroke (width 0) (type default))
-  )
-  (wire (pts (xy 120 46) (xy 116 46))
-    (stroke (width 0) (type default))
-  )
-  (wire (pts (xy 120 50) (xy 116 50))
-    (stroke (width 0) (type default))
-  )
-  (wire (pts (xy 120 54) (xy 116 54))
-    (stroke (width 0) (type default))
-  )
-  (wire (pts (xy 120 58) (xy 116 58))
-    (stroke (width 0) (type default))
-  )
-  (wire (pts (xy 120 62) (xy 116 62))
-    (stroke (width 0) (type default))
-  )
-  (wire (pts (xy 120 66) (xy 116 66))
-    (stroke (width 0) (type default))
-  )
-  (wire (pts (xy 120 70) (xy 116 70))
-    (stroke (width 0) (type default))
-  )
-  (wire (pts (xy 120 74) (xy 116 74))
+  (wire (pts (xy 120 40) (xy 116 40))
+    (stroke (width 0) (type default))
+  )
+  (wire (pts (xy 120 44) (xy 116 44))
+    (stroke (width 0) (type default))
+  )
+  (wire (pts (xy 120 48) (xy 116 48))
+    (stroke (width 0) (type default))
+  )
+  (wire (pts (xy 120 52) (xy 116 52))
+    (stroke (width 0) (type default))
+  )
+  (wire (pts (xy 120 56) (xy 116 56))
+    (stroke (width 0) (type default))
+  )
+  (wire (pts (xy 120 64) (xy 116 64))
+    (stroke (width 0) (type default))
+  )
+  (wire (pts (xy 120 68) (xy 116 68))
+    (stroke (width 0) (type default))
+  )
+  (wire (pts (xy 120 72) (xy 116 72))
     (stroke (width 0) (type default))
   )
@@
     (stroke (width 0) (type default))
   )
-  (wire (pts (xy 88.92 66) (xy 94 66))
-    (stroke (width 0) (type default))
-  )
