File: circuit/kicad/sheet_m0_core_strip.kicad_sch (KiCad schematic)
At the start: 2 parts, among them U201 Feather_M0, U202 NeoPXL8_FeatherWing

Commit message: Migrate Orciny device to single-strip core and GPIO pump control
Replace the M0 NeoPXL8-based core controller with a single 30-pixel NeoPixel strip on D13 and keep Serial1 TX dedicated to RP2040 effect commands.

Replace Motor FeatherWing pump control with direct RP2040 GP8 MOSFET drive while keeping GP7 assigned to the FP-S14B claw servo.

Update both firmware sketches and DeviceConfig headers to match the revised controller responsibilities, serial command flow, and output mappings.

Restructure the KiCad project by removing the legacy NeoPXL8 and motor-and-claw sheets, adding the new core-strip and pump-and-claw sheets, and aligning the block hierarchy and power sheet with the current 5V bus plus 3V filament rail model.

Synchronize README, ASCII wiring, Mermaid wiring, Fritzing mapping, wire labels, KiCad netmaps, and BOM so the documented hardware revision matches the firmware and schematics.

Standardize beam and filament resistor values across the documentation and KiCad sources and retain a compatibility copy of the older KiCad netmap without leaving contradictory power-rail guidance.
Parts:
- J201: renamed from U202; value NeoPXL8_FeatherWing -> Core_Strip; footprint Adafruit_Eagle:FEATHERWING -> Adafruit_Eagle:JST-PH-3-THM; symbol Connector_Generic:Conn_01x12 -> Connector_Generic:Conn_01x03
Other:
- title: Feather M0 + NeoPXL8 -> Feather M0 + Core Strip
Changed lines of the file:
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@@
   (paper "A4")
   (title_block
-    (title "Feather M0 + NeoPXL8")
-    (date "2026-03-30")
-    (rev "B")
+    (title "Feather M0 + Core Strip")
+    (date "2026-03-31")
+    (rev "C")
   )
   (hierarchical_label "SERIAL_LINK" (shape input) (at 20 28 180)
     (effects (font (size 1.27 1.27)) (justify right))
   )
-  (hierarchical_label "+5V_LOGIC" (shape input) (at 20 32 180)
+  (hierarchical_label "+5V_BUS" (shape input) (at 20 32 180)
     (effects (font (size 1.27 1.27)) (justify right))
   )
@@
     (effects (font (size 1.27 1.27)) (justify right))
   )
-  (hierarchical_label "CORE_D0" (shape output) (at 120 44 0)
-    (effects (font (size 1.27 1.27)) (justify left))
-  )
-  (hierarchical_label "CORE_D1" (shape output) (at 120 48 0)
-    (effects (font (size 1.27 1.27)) (justify left))
-  )
-  (hierarchical_label "CORE_D2" (shape output) (at 120 52 0)
-    (effects (font (size 1.27 1.27)) (justify left))
-  )
-  (hierarchical_label "CORE_D3" (shape output) (at 120 56 0)
+  (hierarchical_label "CORE_DATA" (shape output) (at 120 44 0)
     (effects (font (size 1.27 1.27)) (justify left))
   )
@@
     (pin "12")
   )
-  (symbol (lib_id "Connector_Generic:Conn_01x12") (at 84 42 0) (unit 1)
+  (symbol (lib_id "Connector_Generic:Conn_01x03") (at 92 44 0) (unit 1)
     (in_bom yes) (on_board yes)
-    (property "Reference" "U202" (id 0) (at 84 27 0))
-    (property "Value" "NeoPXL8_FeatherWing" (id 1) (at 86.54 42 90))
-    (property "Footprint" "Adafruit_Eagle:FEATHERWING" (id 2) (at 84 42 0)
+    (property "Reference" "J201" (id 0) (at 92 38 0))
+    (property "Value" "Core_Strip" (id 1) (at 94.54 44 90))
+    (property "Footprint" "Adafruit_Eagle:JST-PH-3-THM" (id 2) (at 92 44 0)
       (effects (font (size 1.27 1.27)) hide)
     )
-    (property "Datasheet" "" (id 3) (at 84 42 0))
+    (property "Datasheet" "" (id 3) (at 92 44 0))
     (pin "1")
     (pin "2")
     (pin "3")
-    (pin "4")
-    (pin "5")
-    (pin "6")
-    (pin "7")
-    (pin "8")
-    (pin "9")
-    (pin "10")
-    (pin "11")
-    (pin "12")
   )
   (label "SERIAL_LINK" (at 56.92 28.03 0)
     (effects (font (size 1.27 1.27)) (justify left bottom))
   )
-  (label "+5V_LOGIC" (at 56.92 30.57 0)
+  (label "+5V_BUS" (at 56.92 30.57 0)
     (effects (font (size 1.27 1.27)) (justify left bottom))
   )
@@
     (effects (font (size 1.27 1.27)) (justify left bottom))
   )
-  (label "CORE_D0" (at 78.92 28.03 0)
+  (label "CORE_DATA" (at 78.92 28.03 0)
     (effects (font (size 1.27 1.27)) (justify left bottom))
   )
-  (label "CORE_D1" (at 78.92 30.57 0)
+  (label "CORE_DATA" (at 86.92 42.73 0)
     (effects (font (size 1.27 1.27)) (justify left bottom))
   )
-  (label "CORE_D2" (at 78.92 33.11 0)
+  (label "+5V_BUS" (at 86.92 45.27 0)
     (effects (font (size 1.27 1.27)) (justify left bottom))
   )
-  (label "CORE_D3" (at 78.92 35.65 0)
+  (label "GND_COMMON" (at 86.92 47.81 0)
     (effects (font (size 1.27 1.27)) (justify left bottom))
   )
@@
     (stroke (width 0) (type default))
   )
-  (wire (pts (xy 120 48) (xy 116 48))
-    (stroke (width 0) (type default))
-  )
-  (wire (pts (xy 120 52) (xy 116 52))
-    (stroke (width 0) (type default))
-  )
-  (wire (pts (xy 120 56) (xy 116 56))
-    (stroke (width 0) (type default))
-  )
   (wire (pts (xy 56.92 28.03) (xy 61.5 28.03))
     (stroke (width 0) (type default))
@@
     (stroke (width 0) (type default))
   )
-  (wire (pts (xy 78.92 30.57) (xy 83.5 30.57))
+  (wire (pts (xy 86.92 42.73) (xy 92 42.73))
     (stroke (width 0) (type default))
   )
-  (wire (pts (xy 78.92 33.11) (xy 83.5 33.11))
+  (wire (pts (xy 86.92 45.27) (xy 92 45.27))
     (stroke (width 0) (type default))
   )
-  (wire (pts (xy 78.92 35.65) (xy 83.5 35.65))
+  (wire (pts (xy 86.92 47.81) (xy 92 47.81))
     (stroke (width 0) (type default))
   )
@@
     )
     (path "/e89d3fd8-1532-4ec1-ba22-eb20f36ec0de"
-      (reference "U202") (unit 1) (value "NeoPXL8_FeatherWing") (footprint "Adafruit_Eagle:FEATHERWING")
+      (reference "J201") (unit 1) (value "Core_Strip") (footprint "Adafruit_Eagle:JST-PH-3-THM")
     )
   )

Commit message: Merge Box updates, normalize circuit layout, and add Box sync workflow
Parts:
- U201: value Feather_M0 -> Core_Controller_IO
Other:
- title: Feather M0 + Core Strip -> Core NeoPixel Strip
Changed lines of the file:
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@@
   (paper "A4")
   (title_block
-    (title "Feather M0 + Core Strip")
+    (title "Core NeoPixel Strip")
     (date "2026-03-31")
-    (rev "C")
+    (rev "D")
   )
-  (hierarchical_label "SERIAL_LINK" (shape input) (at 20 28 180)
+  (hierarchical_label "CORE_DATA" (shape input) (at 20 28 180)
     (effects (font (size 1.27 1.27)) (justify right))
   )
@@
     (in_bom yes) (on_board yes)
     (property "Reference" "U201" (id 0) (at 62 27 0))
-    (property "Value" "Feather_M0" (id 1) (at 64.54 42 90))
+    (property "Value" "Core_Controller_IO" (id 1) (at 64.54 42 90))
     (property "Footprint" "Adafruit_Eagle:FEATHERWING" (id 2) (at 62 42 0)
       (effects (font (size 1.27 1.27)) hide)
@@
     (pin "3")
   )
-  (label "SERIAL_LINK" (at 56.92 28.03 0)
+  (label "CORE_DATA" (at 56.92 28.03 0)
     (effects (font (size 1.27 1.27)) (justify left bottom))
   )
@@
   (symbol_instances
     (path "/c5b4f389-cf4f-4e2a-88f6-c5db8e5c4fec"
-      (reference "U201") (unit 1) (value "Feather_M0") (footprint "Adafruit_Eagle:FEATHERWING")
+      (reference "U201") (unit 1) (value "Core_Controller_IO") (footprint "Adafruit_Eagle:FEATHERWING")
     )
     (path "/e89d3fd8-1532-4ec1-ba22-eb20f36ec0de"
