File: circuit/kicad/sheet_pump_and_claw.kicad_sch (KiCad schematic)
At the start: 3 parts, among them J401 Pump_Load, J402 Claw_Stepper, U401 Motor_FeatherWing

Commit message: Migrate Orciny device to single-strip core and GPIO pump control
Replace the M0 NeoPXL8-based core controller with a single 30-pixel NeoPixel strip on D13 and keep Serial1 TX dedicated to RP2040 effect commands.

Replace Motor FeatherWing pump control with direct RP2040 GP8 MOSFET drive while keeping GP7 assigned to the FP-S14B claw servo.

Update both firmware sketches and DeviceConfig headers to match the revised controller responsibilities, serial command flow, and output mappings.

Restructure the KiCad project by removing the legacy NeoPXL8 and motor-and-claw sheets, adding the new core-strip and pump-and-claw sheets, and aligning the block hierarchy and power sheet with the current 5V bus plus 3V filament rail model.

Synchronize README, ASCII wiring, Mermaid wiring, Fritzing mapping, wire labels, KiCad netmaps, and BOM so the documented hardware revision matches the firmware and schematics.

Standardize beam and filament resistor values across the documentation and KiCad sources and retain a compatibility copy of the older KiCad netmap without leaving contradictory power-rail guidance.
Parts:
- removed U401: Motor_FeatherWing, Adafruit_Eagle:FEATHERWING, symbol Connector_Generic:Conn_01x12
- J402: value Claw_Stepper -> Claw_Servo; footprint Adafruit_Eagle:1X04-3.5MM -> Adafruit_Eagle:1X03; symbol Connector_Generic:Conn_01x04 -> Connector_Generic:Conn_01x03
Other:
- title: Motor Wing + Pump + Claw -> Pump + Claw Actuators
Changed lines of the file:
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@@
   (paper "A4")
   (title_block
-    (title "Motor Wing + Pump + Claw")
-    (date "2026-03-30")
-    (rev "B")
+    (title "Pump + Claw Actuators")
+    (date "2026-03-31")
+    (rev "C")
   )
-  (hierarchical_label "I2C_SDA" (shape bidirectional) (at 20 28 180)
+  (hierarchical_label "PUMP_EN" (shape input) (at 20 28 180)
     (effects (font (size 1.27 1.27)) (justify right))
   )
-  (hierarchical_label "I2C_SCL" (shape bidirectional) (at 20 32 180)
+  (hierarchical_label "SERVO_SIG" (shape input) (at 20 32 180)
     (effects (font (size 1.27 1.27)) (justify right))
   )
-  (hierarchical_label "+12V_MAIN" (shape input) (at 20 36 180)
+  (hierarchical_label "+5V_BUS" (shape input) (at 20 36 180)
     (effects (font (size 1.27 1.27)) (justify right))
   )
   (hierarchical_label "GND_COMMON" (shape input) (at 20 40 180)
     (effects (font (size 1.27 1.27)) (justify right))
-  )
-  (hierarchical_label "M1_PUMP" (shape output) (at 120 48 0)
-    (effects (font (size 1.27 1.27)) (justify left))
-  )
-  (hierarchical_label "STEPPER_P2" (shape output) (at 120 52 0)
-    (effects (font (size 1.27 1.27)) (justify left))
-  )
-  (symbol (lib_id "Connector_Generic:Conn_01x12") (at 60 40 0) (unit 1)
-    (in_bom yes) (on_board yes)
-    (property "Reference" "U401" (id 0) (at 60 25 0))
-    (property "Value" "Motor_FeatherWing" (id 1) (at 62.54 40 90))
-    (property "Footprint" "Adafruit_Eagle:FEATHERWING" (id 2) (at 60 40 0)
-      (effects (font (size 1.27 1.27)) hide)
-    )
-    (property "Datasheet" "" (id 3) (at 60 40 0))
-    (pin "1")
-    (pin "2")
-    (pin "3")
-    (pin "4")
-    (pin "5")
-    (pin "6")
-    (pin "7")
-    (pin "8")
-    (pin "9")
-    (pin "10")
-    (pin "11")
-    (pin "12")
   )
   (symbol (lib_id "Connector_Generic:Conn_01x02") (at 92 44 0) (unit 1)
@@
     (pin "2")
   )
-  (symbol (lib_id "Connector_Generic:Conn_01x04") (at 92 56 0) (unit 1)
+  (symbol (lib_id "Connector_Generic:Conn_01x03") (at 92 56 0) (unit 1)
     (in_bom yes) (on_board yes)
-    (property "Reference" "J402" (id 0) (at 92 49 0))
-    (property "Value" "Claw_Stepper" (id 1) (at 94.54 56 90))
-    (property "Footprint" "Adafruit_Eagle:1X04-3.5MM" (id 2) (at 92 56 0)
+    (property "Reference" "J402" (id 0) (at 92 50 0))
+    (property "Value" "Claw_Servo" (id 1) (at 94.54 56 90))
+    (property "Footprint" "Adafruit_Eagle:1X03" (id 2) (at 92 56 0)
       (effects (font (size 1.27 1.27)) hide)
     )
@@
     (pin "2")
     (pin "3")
-    (pin "4")
   )
-  (label "I2C_SDA" (at 54.92 26.03 0)
+  (label "PUMP_EN" (at 54.92 26.03 0)
     (effects (font (size 1.27 1.27)) (justify left bottom))
   )
-  (label "I2C_SCL" (at 54.92 28.57 0)
+  (label "SERVO_SIG" (at 54.92 28.57 0)
     (effects (font (size 1.27 1.27)) (justify left bottom))
   )
-  (label "+12V_MAIN" (at 54.92 31.11 0)
+  (label "+5V_BUS" (at 54.92 31.11 0)
     (effects (font (size 1.27 1.27)) (justify left bottom))
   )
@@
     (effects (font (size 1.27 1.27)) (justify left bottom))
   )
-  (label "M1_PUMP" (at 54.92 36.19 0)
-    (effects (font (size 1.27 1.27)) (justify left bottom))
-  )
-  (label "STEPPER_P2" (at 54.92 38.73 0)
-    (effects (font (size 1.27 1.27)) (justify left bottom))
-  )
-  (label "M1_PUMP" (at 86.92 42.73 0)
+  (label "PUMP_EN" (at 86.92 42.73 0)
     (effects (font (size 1.27 1.27)) (justify left bottom))
   )
@@
     (effects (font (size 1.27 1.27)) (justify left bottom))
   )
-  (label "STEPPER_P2" (at 86.92 52.19 0)
+  (label "SERVO_SIG" (at 86.92 52.19 0)
     (effects (font (size 1.27 1.27)) (justify left bottom))
   )
-  (label "+12V_MAIN" (at 86.92 54.73 0)
+  (label "+5V_BUS" (at 86.92 54.73 0)
     (effects (font (size 1.27 1.27)) (justify left bottom))
   )
@@
     (stroke (width 0) (type default))
   )
-  (wire (pts (xy 120 48) (xy 116 48))
-    (stroke (width 0) (type default))
-  )
-  (wire (pts (xy 120 52) (xy 116 52))
-    (stroke (width 0) (type default))
-  )
   (wire (pts (xy 54.92 26.03) (xy 60 26.03))
     (stroke (width 0) (type default))
@@
   )
   (wire (pts (xy 54.92 33.65) (xy 60 33.65))
-    (stroke (width 0) (type default))
-  )
-  (wire (pts (xy 54.92 36.19) (xy 60 36.19))
-    (stroke (width 0) (type default))
-  )
-  (wire (pts (xy 54.92 38.73) (xy 60 38.73))
     (stroke (width 0) (type default))
   )
@@
   )
   (symbol_instances
-    (path "/3afb663a-90d4-42d2-87c5-4f6322efde07"
-      (reference "U401") (unit 1) (value "Motor_FeatherWing") (footprint "Adafruit_Eagle:FEATHERWING")
-    )
     (path "/4705ff58-3da2-47f4-9220-989d1451d837"
       (reference "J401") (unit 1) (value "Pump_Load") (footprint "Adafruit_Eagle:JST-PH-2-THM")
     )
     (path "/7214372d-f7ce-4e8f-b299-5a7d9d30ec20"
-      (reference "J402") (unit 1) (value "Claw_Stepper") (footprint "Adafruit_Eagle:1X04-3.5MM")
+      (reference "J402") (unit 1) (value "Claw_Servo") (footprint "Adafruit_Eagle:1X03")
     )
   )

Commit message: Merge Box updates, normalize circuit layout, and add Box sync workflow
Parts:
- added J403: Servo_B, Adafruit_Eagle:JSTPH3, symbol Connector_Generic:Conn_01x03
- J401: value Pump_Load -> Optional_Pump
- J402: value Claw_Servo -> Servo_A; footprint Adafruit_Eagle:1X03 -> Adafruit_Eagle:JSTPH3
Other:
- note added: "PCA9685 servo function on the FeatherWing side CH0 -> Servo_A, CH1 -> Servo_B Pump path is optional and disabled in current firmware"
- title: Pump + Claw Actuators -> Servo FeatherWing + Optional Pump
Changed lines of the file:
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@@
   (paper "A4")
   (title_block
-    (title "Pump + Claw Actuators")
-    (date "2026-03-31")
-    (rev "C")
+    (title "Servo FeatherWing + Optional Pump")
+    (date "2026-04-08")
+    (rev "D")
   )
-  (hierarchical_label "PUMP_EN" (shape input) (at 20 28 180)
+  (hierarchical_label "PUMP_EN_OPTIONAL" (shape input) (at 20 24 180)
     (effects (font (size 1.27 1.27)) (justify right))
   )
-  (hierarchical_label "SERVO_SIG" (shape input) (at 20 32 180)
+  (hierarchical_label "I2C_SDA_SERVO_WING" (shape input) (at 20 28 180)
+    (effects (font (size 1.27 1.27)) (justify right))
+  )
+  (hierarchical_label "I2C_SCL_SERVO_WING" (shape input) (at 20 32 180)
     (effects (font (size 1.27 1.27)) (justify right))
   )
@@
     (effects (font (size 1.27 1.27)) (justify right))
   )
+  (hierarchical_label "SERVO_A_SIG" (shape output) (at 120 54 0)
+    (effects (font (size 1.27 1.27)) (justify left))
+  )
+  (hierarchical_label "SERVO_B_SIG" (shape output) (at 120 58 0)
+    (effects (font (size 1.27 1.27)) (justify left))
+  )
   (symbol (lib_id "Connector_Generic:Conn_01x02") (at 92 44 0) (unit 1)
     (in_bom yes) (on_board yes)
     (property "Reference" "J401" (id 0) (at 92 39 0))
-    (property "Value" "Pump_Load" (id 1) (at 94.54 44 90))
+    (property "Value" "Optional_Pump" (id 1) (at 94.54 44 90))
     (property "Footprint" "Adafruit_Eagle:JST-PH-2-THM" (id 2) (at 92 44 0)
       (effects (font (size 1.27 1.27)) hide)
@@
     (in_bom yes) (on_board yes)
     (property "Reference" "J402" (id 0) (at 92 50 0))
-    (property "Value" "Claw_Servo" (id 1) (at 94.54 56 90))
-    (property "Footprint" "Adafruit_Eagle:1X03" (id 2) (at 92 56 0)
+    (property "Value" "Servo_A" (id 1) (at 94.54 56 90))
+    (property "Footprint" "Adafruit_Eagle:JSTPH3" (id 2) (at 92 56 0)
       (effects (font (size 1.27 1.27)) hide)
     )
@@
     (pin "3")
   )
-  (label "PUMP_EN" (at 54.92 26.03 0)
+  (symbol (lib_id "Connector_Generic:Conn_01x03") (at 110 56 0) (unit 1)
+    (in_bom yes) (on_board yes)
+    (property "Reference" "J403" (id 0) (at 110 50 0))
+    (property "Value" "Servo_B" (id 1) (at 112.54 56 90))
+    (property "Footprint" "Adafruit_Eagle:JSTPH3" (id 2) (at 110 56 0)
+      (effects (font (size 1.27 1.27)) hide)
+    )
+    (property "Datasheet" "" (id 3) (at 110 56 0))
+    (pin "1")
+    (pin "2")
+    (pin "3")
+  )
+  (text "PCA9685 servo function on the FeatherWing side\nCH0 -> Servo_A, CH1 -> Servo_B\nPump path is optional and disabled in current firmware" (at 56 18 0)
+    (effects (font (size 1.27 1.27)) (justify left top))
+  )
+  (label "PUMP_EN_OPTIONAL" (at 54.92 23.49 0)
     (effects (font (size 1.27 1.27)) (justify left bottom))
   )
-  (label "SERVO_SIG" (at 54.92 28.57 0)
+  (label "I2C_SDA_SERVO_WING" (at 54.92 26.03 0)
+    (effects (font (size 1.27 1.27)) (justify left bottom))
+  )
+  (label "I2C_SCL_SERVO_WING" (at 54.92 28.57 0)
     (effects (font (size 1.27 1.27)) (justify left bottom))
   )
@@
     (effects (font (size 1.27 1.27)) (justify left bottom))
   )
-  (label "PUMP_EN" (at 86.92 42.73 0)
+  (label "PUMP_EN_OPTIONAL" (at 86.92 42.73 0)
     (effects (font (size 1.27 1.27)) (justify left bottom))
   )
@@
     (effects (font (size 1.27 1.27)) (justify left bottom))
   )
-  (label "SERVO_SIG" (at 86.92 52.19 0)
+  (label "SERVO_A_SIG" (at 86.92 52.19 0)
     (effects (font (size 1.27 1.27)) (justify left bottom))
   )
@@
   (label "GND_COMMON" (at 86.92 57.27 0)
     (effects (font (size 1.27 1.27)) (justify left bottom))
+  )
+  (label "SERVO_B_SIG" (at 104.92 52.19 0)
+    (effects (font (size 1.27 1.27)) (justify left bottom))
+  )
+  (label "+5V_BUS" (at 104.92 54.73 0)
+    (effects (font (size 1.27 1.27)) (justify left bottom))
+  )
+  (label "GND_COMMON" (at 104.92 57.27 0)
+    (effects (font (size 1.27 1.27)) (justify left bottom))
+  )
+  (wire (pts (xy 20 24) (xy 24 24))
+    (stroke (width 0) (type default))
   )
   (wire (pts (xy 20 28) (xy 24 28))
@@
   )
   (wire (pts (xy 20 40) (xy 24 40))
+    (stroke (width 0) (type default))
+  )
+  (wire (pts (xy 54.92 23.49) (xy 60 23.49))
     (stroke (width 0) (type default))
   )
@@
     (stroke (width 0) (type default))
   )
+  (wire (pts (xy 104.92 52.19) (xy 110 52.19))
+    (stroke (width 0) (type default))
+  )
+  (wire (pts (xy 104.92 54.73) (xy 110 54.73))
+    (stroke (width 0) (type default))
+  )
+  (wire (pts (xy 104.92 57.27) (xy 110 57.27))
+    (stroke (width 0) (type default))
+  )
+  (wire (pts (xy 116 54) (xy 120 54))
+    (stroke (width 0) (type default))
+  )
+  (wire (pts (xy 116 58) (xy 120 58))
+    (stroke (width 0) (type default))
+  )
   (sheet_instances
     (path "/" (page "4"))
@@
   (symbol_instances
     (path "/4705ff58-3da2-47f4-9220-989d1451d837"
-      (reference "J401") (unit 1) (value "Pump_Load") (footprint "Adafruit_Eagle:JST-PH-2-THM")
+      (reference "J401") (unit 1) (value "Optional_Pump") (footprint "Adafruit_Eagle:JST-PH-2-THM")
     )
     (path "/7214372d-f7ce-4e8f-b299-5a7d9d30ec20"
-      (reference "J402") (unit 1) (value "Claw_Servo") (footprint "Adafruit_Eagle:1X03")
+      (reference "J402") (unit 1) (value "Servo_A") (footprint "Adafruit_Eagle:JSTPH3")
+    )
+    (path "/24932f34-3552-48ae-9327-a94e6555da0e"
+      (reference "J403") (unit 1) (value "Servo_B") (footprint "Adafruit_Eagle:JSTPH3")
     )
   )
