File: circuit/kicad/sheet_switches.kicad_sch (KiCad schematic)
At the start: 3 parts, among them SW1 SW_Toggle, SW2 SW_Prev, SW3 SW_Next

Commit message: Merge Box updates, normalize circuit layout, and add Box sync workflow
Parts:
- renumbered SW3 to SW?, SW2 to SW?, SW1 to SW?
